Commit message: Fixed joints

File: body.urdf (robot description, URDF)
Before this commit: robot robot, 3 links, 2 joints
Joints:
- joint Torso_BackLeg: origin xyz=0 0 1 rpy=0 0 0 -> xyz=-0.5 0 1 rpy=0 0 0
- joint Torso_FrontLeg: origin xyz=0 0 1 rpy=0 0 0 -> xyz=0.5 0 1 rpy=0 0 0

Commit message: Finished :)

File: body.urdf (robot description, URDF)
Before this commit: robot robot, 3 links, 2 joints
Links:
- added link LeftLeg, mass 1; collision box size=1 0.2 0.2; visual box size=1 0.2 0.2
- added link LowerBaLeg, mass 1; collision box size=0.2 0.2 1; visual box size=0.2 0.2 1
- added link LowerFrLeg, mass 1; collision box size=0.2 0.2 1; visual box size=0.2 0.2 1
- added link LowerLeLeg, mass 1; collision box size=0.2 0.2 1; visual box size=0.2 0.2 1
- added link LowerRiLeg, mass 1; collision box size=0.2 0.2 1; visual box size=0.2 0.2 1
- added link RightLeg, mass 1; collision box size=1 0.2 0.2; visual box size=1 0.2 0.2
- link BackLeg: geometry collision box size=0.2 1 0.2; visual box size=0.2 1 0.2
- link FrontLeg: geometry collision box size=0.2 1 0.2; visual box size=0.2 1 0.2
Joints:
- added joint BackLeg_LowerBaLeg: type revolute, parent BackLeg, child LowerBaLeg, origin xyz=0 -1 0 rpy=0 0 0, axis 1 0 0, limit lower=-3.14159 upper=3.14159 effort=0.0 velocity=0.0
- added joint FrontLeg_LowerFrLeg: type revolute, parent FrontLeg, child LowerFrLeg, origin xyz=0 1 0 rpy=0 0 0, axis 1 0 0, limit lower=-3.14159 upper=3.14159 effort=0.0 velocity=0.0
- added joint LeftLeg_LowerLeLeg: type revolute, parent LeftLeg, child LowerLeLeg, origin xyz=1 0 0 rpy=0 0 0, axis 0 1 0, limit lower=-3.14159 upper=3.14159 effort=0.0 velocity=0.0
- added joint RightLeg_LowerRiLeg: type revolute, parent RightLeg, child LowerRiLeg, origin xyz=-1 0 0 rpy=0 0 0, axis 0 1 0, limit lower=-3.14159 upper=3.14159 effort=0.0 velocity=0.0
- added joint Torso_LeftLeg: type revolute, parent Torso, child LeftLeg, origin xyz=0.5 0 1 rpy=0 0 0, axis 0 1 0, limit lower=-3.14159 upper=3.14159 effort=0.0 velocity=0.0
- added joint Torso_RightLeg: type revolute, parent Torso, child RightLeg, origin xyz=-0.5 0 1 rpy=0 0 0, axis 0 1 0, limit lower=-3.14159 upper=3.14159 effort=0.0 velocity=0.0
- joint Torso_BackLeg: axis 0 1 0 -> 1 0 0; origin xyz=-0.5 0 1 rpy=0 0 0 -> xyz=0 -0.5 1 rpy=0 0 0
- joint Torso_FrontLeg: axis 0 1 0 -> 1 0 0; origin xyz=0.5 0 1 rpy=0 0 0 -> xyz=0 0.5 1 rpy=0 0 0

Commit message: Does not work yet

File: body.urdf (robot description, URDF)
Before this commit: robot robot, 9 links, 8 joints
Links:
- removed link BackLeg
- removed link FrontLeg
- removed link LeftLeg
- removed link LowerBaLeg
- removed link LowerFrLeg
- removed link LowerLeLeg
- removed link LowerRiLeg
- removed link RightLeg
- removed link Torso
- added link Link1, mass 1; collision box size=3 2 0.5; visual box size=3 2 0.5
- added link Link2, mass 1; collision box size=0.25 1.75 0.5; visual box size=0.25 1.75 0.5
- added link Link3, mass 1; collision box size=1 4 0.5; visual box size=1 4 0.5
- added link Tracker, mass 1; collision box size=0.25 0.25 0.5; visual box size=0.25 0.25 0.5
- added link Wheel1, mass 1; collision sphere radius=0.5; visual sphere radius=0.5
- added link Wheel2, mass 1; collision sphere radius=0.5; visual sphere radius=0.5
- added link Wheel3, mass 1; collision sphere radius=0.5; visual sphere radius=0.5
Joints:
- removed joint BackLeg_LowerBaLeg
- removed joint FrontLeg_LowerFrLeg
- removed joint LeftLeg_LowerLeLeg
- removed joint RightLeg_LowerRiLeg
- removed joint Torso_BackLeg
- removed joint Torso_FrontLeg
- removed joint Torso_LeftLeg
- removed joint Torso_RightLeg
- added joint Link1_Link2: type fixed, parent Link1, child Link2, origin xyz=1.5 0 1.25 rpy=0 0 0, axis 0 1 0, limit lower=-3.14159 upper=3.14159 effort=1.0 velocity=0.0
- added joint Link1_Wheel1: type continuous, parent Link1, child Wheel1, origin xyz=-0.75 0 1 rpy=0 0 0, axis 0 1 0, limit lower=-3.14159 upper=3.14159 effort=1.0 velocity=0.0
- added joint Link2_Link3: type fixed, parent Link2, child Link3, origin xyz=0.25 0 0 rpy=0 0 0, axis 0 1 0, limit lower=-3.14159 upper=3.14159 effort=1.0 velocity=0.0
- added joint Link2_Tracker: type fixed, parent Link2, child Tracker, origin xyz=0.125 0.75 0 rpy=0 0 0, axis 0 1 0, limit lower=-3.14159 upper=3.14159 effort=1.0 velocity=0.0
- added joint Link3_Wheel2: type fixed, parent Link3, child Wheel2, origin xyz=0.5 2.5 -0.25 rpy=0 0 0, axis 0 1 0, limit lower=-3.14159 upper=3.14159 effort=1.0 velocity=0.0
- added joint Link3_Wheel3: type continuous, parent Link3, child Wheel3, origin xyz=0.5 0 -0.25 rpy=0 0 0, axis 1 0 0, limit lower=-3.14159 upper=3.14159 effort=1.0 velocity=0.0

Commit message: kinda working

File: body.urdf (robot description, URDF)
Before this commit: robot robot, 9 links, 8 joints
Links:
- removed link BackLeg
- removed link FrontLeg
- removed link LeftLeg
- removed link LowerBaLeg
- removed link LowerFrLeg
- removed link LowerLeLeg
- removed link LowerRiLeg
- removed link RightLeg
- removed link Torso
- added link Leg1Lower, mass 1; collision box size=0.3 0.3 1; visual box size=0.3 0.3 1
- added link Leg1Upper, mass 1; collision box size=0.5 0.5 1; visual box size=0.5 0.5 1
- added link Leg2Lower, mass 1; collision box size=0.3 0.3 1; visual box size=0.3 0.3 1
- added link Leg2Upper, mass 1; collision box size=0.5 0.5 1; visual box size=0.5 0.5 1
- added link Leg3Lower, mass 1; collision box size=0.3 0.3 1; visual box size=0.3 0.3 1
- added link Leg3Upper, mass 1; collision box size=0.5 0.5 1; visual box size=0.5 0.5 1
- added link Link1, mass 1; collision box size=3 2 0.5; visual box size=3 2 0.5
- added link Link2, mass 1; collision box size=0.25 1.75 0.5; visual box size=0.25 1.75 0.5
- added link Link3, mass 1; collision box size=1 4 0.5; visual box size=1 4 0.5
- added link Tracker, mass 1; collision box size=0.25 0.25 0.5; visual box size=0.25 0.25 0.5
Joints:
- removed joint BackLeg_LowerBaLeg
- removed joint FrontLeg_LowerFrLeg
- removed joint LeftLeg_LowerLeLeg
- removed joint RightLeg_LowerRiLeg
- removed joint Torso_BackLeg
- removed joint Torso_FrontLeg
- removed joint Torso_LeftLeg
- removed joint Torso_RightLeg
- added joint Leg1Upper_Leg1Lower: type revolute, parent Leg1Upper, child Leg1Lower, origin xyz=0 0 -1 rpy=0 0 0, axis 0 1 0, limit lower=-3.14159 upper=3.14159 effort=0.0 velocity=0.0
- added joint Leg2Upper_Leg2Lower: type revolute, parent Leg2Upper, child Leg2Lower, origin xyz=0 0 -1 rpy=0 0 0, axis 0 1 0, limit lower=-3.14159 upper=3.14159 effort=0.0 velocity=0.0
- added joint Leg3Upper_Leg3Lower: type revolute, parent Leg3Upper, child Leg3Lower, origin xyz=0 0 -1 rpy=0 0 0, axis 0 1 0, limit lower=-3.14159 upper=3.14159 effort=0.0 velocity=0.0
- added joint Link1_Leg1Upper: type revolute, parent Link1, child Leg1Upper, origin xyz=-1.5 0 2.25 rpy=0 0 0, axis 0 1 0, limit lower=-3.14159 upper=3.14159 effort=0.0 velocity=0.0
- added joint Link1_Link2: type fixed, parent Link1, child Link2, origin xyz=1.5 0 2.25 rpy=0 0 0, axis 0 1 0, limit lower=-3.14159 upper=3.14159 effort=0.0 velocity=0.0
- added joint Link2_Link3: type fixed, parent Link2, child Link3, origin xyz=0.25 0 0 rpy=0 0 0, axis 0 1 0, limit lower=-3.14159 upper=3.14159 effort=0.0 velocity=0.0
- added joint Link2_Tracker: type fixed, parent Link2, child Tracker, origin xyz=0.125 0.75 0 rpy=0 0 0, axis 0 1 0, limit lower=-3.14159 upper=3.14159 effort=0.0 velocity=0.0
- added joint Link3_Leg2Upper: type revolute, parent Link3, child Leg2Upper, origin xyz=1 0 0 rpy=0 0 0, axis 0 1 0, limit lower=-3.14159 upper=3.14159 effort=0.0 velocity=0.0
- added joint Link3_Leg3Upper: type revolute, parent Link3, child Leg3Upper, origin xyz=1 2 0 rpy=0 0 0, axis 0 1 0, limit lower=-3.14159 upper=3.14159 effort=0.0 velocity=0.0

Commit message: Finished?

File: body.urdf (robot description, URDF)
Before this commit: robot robot, 10 links, 9 joints
Joints:
- joint Leg2Upper_Leg2Lower: axis 0 1 0 -> 1 0 0
- joint Link3_Leg2Upper: axis 0 1 0 -> 1 0 0

Commit message: Finished functional motors :D

File: body.urdf (robot description, URDF)
Before this commit: robot robot, 10 links, 9 joints
Joints:
- joint Leg2Upper_Leg2Lower: axis 1 0 0 -> 0 1 0
- joint Link3_Leg2Upper: axis 1 0 0 -> 0 1 0

File: snake.urdf (robot description, URDF)
Before this commit: robot robot, 15 links, 14 joints
Links:
- removed link 10
- removed link 11
- removed link 12
- removed link 13
- removed link 14
- removed link 5
- removed link 6
- removed link 7
- removed link 8
- removed link 9
- link 0: geometry collision box size=0.841986828690744 0.6562646693395983 1.2500115242528775; visual box size=0.841986828690744 0.6562646693395983 1.2500115242528775
- link 1: geometry collision box size=0.8382508003398526 0.7089643006462857 0.7055372258848194; visual box size=0.8382508003398526 0.7089643006462857 0.7055372258848194
- link 2: geometry collision box size=1.0966477965233212 0.10836637661855801 1.2416623520251409; visual box size=1.0966477965233212 0.10836637661855801 1.2416623520251409
- link 3: geometry collision box size=1.1596397643018466 0.6500876888342165 0.5366664630718985; visual box size=1.1596397643018466 0.6500876888342165 0.5366664630718985
- link 4: geometry collision box size=0.8814621431917291 0.3992100740515573 0.4088639618745678; visual box size=0.8814621431917291 0.3992100740515573 0.4088639618745678
Joints:
- removed joint 10_11
- removed joint 11_12
- removed joint 12_13
- removed joint 13_14
- removed joint 4_5
- removed joint 5_6
- removed joint 6_7
- removed joint 7_8
- removed joint 8_9
- removed joint 9_10
- joint 0_1: axis 0 0 1 -> 0 1 0; origin xyz=0.5771985920131326 0 5 rpy=0 0 0 -> xyz=0.420993414345372 0 5 rpy=0 0 0
- joint 1_2: origin xyz=1.64955015919415 0 0 rpy=0 0 0 -> xyz=0.8382508003398526 0 0 rpy=0 0 0
- joint 2_3: axis 0 0 1 -> 0 1 0; origin xyz=1.6842005734744627 0 0 rpy=0 0 0 -> xyz=1.0966477965233212 0 0 rpy=0 0 0
- joint 3_4: axis 0 1 0 -> 0 0 1; origin xyz=1.435140497289197 0 0 rpy=0 0 0 -> xyz=1.1596397643018466 0 0 rpy=0 0 0
