Commit message: Generating the morphology!

File: snake.urdf (robot description, URDF)
Before this commit: robot robot, 5 links, 4 joints
Links:
- link 0: geometry collision box size=0.8036591950497327 0.9076406529671176 0.8167793728116315; visual box size=0.8036591950497327 0.9076406529671176 0.8167793728116315
- link 1: geometry collision box size=0.8428604288650012 0.7973259130979675 0.7713723722547201; visual box size=0.8428604288650012 0.7973259130979675 0.7713723722547201
- link 2: geometry collision box size=0.7629162181349561 0.8754775673539389 0.9894469775026211; visual box size=0.7629162181349561 0.8754775673539389 0.9894469775026211
- link 3: geometry collision box size=0.9979057292382096 0.9166268309334646 0.9872583484862485; visual box size=0.9979057292382096 0.9166268309334646 0.9872583484862485
- link 4: geometry collision box size=0.9806095745459124 0.9708871686721723 0.7896178541604109; visual box size=0.9806095745459124 0.9708871686721723 0.7896178541604109
Joints:
- joint 0_1: axis 0 0 1 -> 0 1 0; origin xyz=0.8277634063454427 0 5 rpy=0 0 0 -> xyz=0.8036591950497327 0 5 rpy=0 0 0
- joint 1_2: axis 0 0 1 -> 0 1 0; origin xyz=0.9757676619844111 0 5 rpy=0 0 0 -> xyz=0.8428604288650012 0 5 rpy=0 0 0
- joint 2_3: axis 0 1 0 -> 0 0 1; origin xyz=0.9406366986398206 0 5 rpy=0 0 0 -> xyz=0.7629162181349561 0 5 rpy=0 0 0
- joint 3_4: axis 0 1 0 -> 0 0 1; origin xyz=0.7572163685526483 0 5 rpy=0 0 0 -> xyz=0.9979057292382096 0 5 rpy=0 0 0

Commit message: Fully random morphology :)

File: snake.urdf (robot description, URDF)
Before this commit: robot robot, 5 links, 4 joints
Links:
- added link 10, mass 1; collision box size=1.2432014684837993 0.10553680334614504 1.2361189300063091; visual box size=1.2432014684837993 0.10553680334614504 1.2361189300063091
- added link 11, mass 1; collision box size=1.6176582042089012 0.8171030189291146 0.6669029611488054; visual box size=1.6176582042089012 0.8171030189291146 0.6669029611488054
- added link 12, mass 1; collision box size=1.6230898241782483 0.9002637214467127 0.3790585427471542; visual box size=1.6230898241782483 0.9002637214467127 0.3790585427471542
- added link 13, mass 1; collision box size=1.8280689711247264 1.4415967896302548 0.5236145074472098; visual box size=1.8280689711247264 1.4415967896302548 0.5236145074472098
- added link 14, mass 1; collision box size=1.7013433623433192 0.7534878885286235 0.8572446809719734; visual box size=1.7013433623433192 0.7534878885286235 0.8572446809719734
- added link 5, mass 1; collision box size=0.9715559888863767 0.7026680844571941 0.8307956645081632; visual box size=0.9715559888863767 0.7026680844571941 0.8307956645081632
- added link 6, mass 1; collision box size=1.4021930467757744 0.6083579600181905 0.8534030362153102; visual box size=1.4021930467757744 0.6083579600181905 0.8534030362153102
- added link 7, mass 1; collision box size=1.3072611770680513 0.5813781376856125 0.581956948114435; visual box size=1.3072611770680513 0.5813781376856125 0.581956948114435
- added link 8, mass 1; collision box size=1.2429960486923146 0.7877818155369603 0.48573963331306624; visual box size=1.2429960486923146 0.7877818155369603 0.48573963331306624
- added link 9, mass 1; collision box size=1.6117234382669712 0.5441743691971781 0.4651607790749181; visual box size=1.6117234382669712 0.5441743691971781 0.4651607790749181
- link 0: geometry collision box size=1.1543971840262652 0.04429404614026686 0.2625731593245; visual box size=1.1543971840262652 0.04429404614026686 0.2625731593245
- link 1: geometry collision box size=1.64955015919415 0.40468093876798134 0.7618054619732614; visual box size=1.64955015919415 0.40468093876798134 0.7618054619732614
- link 2: geometry collision box size=1.6842005734744627 0.1616816730676489 0.37582688022141936; visual box size=1.6842005734744627 0.1616816730676489 0.37582688022141936
- link 3: geometry collision box size=1.435140497289197 0.9667606291234939 0.12014328402893631; visual box size=1.435140497289197 0.9667606291234939 0.12014328402893631
- link 4: geometry collision box size=0.9493500493977466 0.5875457101811637 1.0224578553879506; visual box size=0.9493500493977466 0.5875457101811637 1.0224578553879506
Joints:
- added joint 10_11: type revolute, parent 10, child 11, origin xyz=1.2432014684837993 0 0 rpy=0 0 0, axis 0 1 0, limit lower=-3.14159 upper=3.14159 effort=0.0 velocity=0.0
- added joint 11_12: type revolute, parent 11, child 12, origin xyz=1.6176582042089012 0 0 rpy=0 0 0, axis 0 1 0, limit lower=-3.14159 upper=3.14159 effort=0.0 velocity=0.0
- added joint 12_13: type revolute, parent 12, child 13, origin xyz=1.6230898241782483 0 0 rpy=0 0 0, axis 0 1 0, limit lower=-3.14159 upper=3.14159 effort=0.0 velocity=0.0
- added joint 13_14: type revolute, parent 13, child 14, origin xyz=1.8280689711247264 0 0 rpy=0 0 0, axis 0 1 0, limit lower=-3.14159 upper=3.14159 effort=0.0 velocity=0.0
- added joint 4_5: type revolute, parent 4, child 5, origin xyz=0.9493500493977466 0 0 rpy=0 0 0, axis 0 0 1, limit lower=-3.14159 upper=3.14159 effort=0.0 velocity=0.0
- added joint 5_6: type revolute, parent 5, child 6, origin xyz=0.9715559888863767 0 0 rpy=0 0 0, axis 0 0 1, limit lower=-3.14159 upper=3.14159 effort=0.0 velocity=0.0
- added joint 6_7: type revolute, parent 6, child 7, origin xyz=1.4021930467757744 0 0 rpy=0 0 0, axis 0 0 1, limit lower=-3.14159 upper=3.14159 effort=0.0 velocity=0.0
- added joint 7_8: type revolute, parent 7, child 8, origin xyz=1.3072611770680513 0 0 rpy=0 0 0, axis 0 1 0, limit lower=-3.14159 upper=3.14159 effort=0.0 velocity=0.0
- added joint 8_9: type revolute, parent 8, child 9, origin xyz=1.2429960486923146 0 0 rpy=0 0 0, axis 0 1 0, limit lower=-3.14159 upper=3.14159 effort=0.0 velocity=0.0
- added joint 9_10: type revolute, parent 9, child 10, origin xyz=1.6117234382669712 0 0 rpy=0 0 0, axis 0 0 1, limit lower=-3.14159 upper=3.14159 effort=0.0 velocity=0.0
- joint 0_1: axis 0 1 0 -> 0 0 1; origin xyz=0.8036591950497327 0 5 rpy=0 0 0 -> xyz=0.5771985920131326 0 5 rpy=0 0 0
- joint 1_2: axis 0 1 0 -> 0 0 1; origin xyz=0.8428604288650012 0 5 rpy=0 0 0 -> xyz=1.64955015919415 0 0 rpy=0 0 0
- joint 2_3: origin xyz=0.7629162181349561 0 5 rpy=0 0 0 -> xyz=1.6842005734744627 0 0 rpy=0 0 0
- joint 3_4: axis 0 0 1 -> 0 1 0; origin xyz=0.9979057292382096 0 5 rpy=0 0 0 -> xyz=1.435140497289197 0 0 rpy=0 0 0

Commit message: Changing constants

File: snake.urdf (robot description, URDF)
Before this commit: robot robot, 5 links, 4 joints
Links:
- added link 10, mass 1; collision box size=1.1443524188494578 1.171046386485654 0.7855643014504557; visual box size=1.1443524188494578 1.171046386485654 0.7855643014504557
- added link 5, mass 1; collision box size=0.895085736659456 1.3905656148282124 0.8376599325116689; visual box size=0.895085736659456 1.3905656148282124 0.8376599325116689
- added link 6, mass 1; collision box size=1.3347876085912813 0.37247280361736856 0.418738414801258; visual box size=1.3347876085912813 0.37247280361736856 0.418738414801258
- added link 7, mass 1; collision box size=0.8837880941459109 1.1712794706936644 0.7099577746228405; visual box size=0.8837880941459109 1.1712794706936644 0.7099577746228405
- added link 8, mass 1; collision box size=1.0269869044018236 0.7903251494368853 0.5465547583489466; visual box size=1.0269869044018236 0.7903251494368853 0.5465547583489466
- added link 9, mass 1; collision box size=0.8489169791059855 0.5381469653884196 0.31459886834177647; visual box size=0.8489169791059855 0.5381469653884196 0.31459886834177647
- link 0: geometry collision box size=0.7705754847940746 0.5885090509659645 1.005734338863237; visual box size=0.7705754847940746 0.5885090509659645 1.005734338863237
- link 1: geometry collision box size=1.176199397605837 0.8357211415970165 0.880680286484615; visual box size=1.176199397605837 0.8357211415970165 0.880680286484615
- link 2: geometry collision box size=1.3958249340268583 1.2218236794581232 0.8379083242673157; visual box size=1.3958249340268583 1.2218236794581232 0.8379083242673157
- link 3: geometry collision box size=0.9883456458746409 0.49674896783433053 0.19238142026008462; visual box size=0.9883456458746409 0.49674896783433053 0.19238142026008462
- link 4: geometry collision box size=1.2269315784281258 0.39963196249023547 0.37245272035683974; visual box size=1.2269315784281258 0.39963196249023547 0.37245272035683974
Joints:
- added joint 4_5: type revolute, parent 4, child 5, origin xyz=1.2269315784281258 0 0 rpy=0 0 0, axis 0 0 1, limit lower=-3.14159 upper=3.14159 effort=0.0 velocity=0.0
- added joint 5_6: type revolute, parent 5, child 6, origin xyz=0.895085736659456 0 0 rpy=0 0 0, axis 0 1 0, limit lower=-3.14159 upper=3.14159 effort=0.0 velocity=0.0
- added joint 6_7: type revolute, parent 6, child 7, origin xyz=1.3347876085912813 0 0 rpy=0 0 0, axis 0 1 0, limit lower=-3.14159 upper=3.14159 effort=0.0 velocity=0.0
- added joint 7_8: type revolute, parent 7, child 8, origin xyz=0.8837880941459109 0 0 rpy=0 0 0, axis 0 1 0, limit lower=-3.14159 upper=3.14159 effort=0.0 velocity=0.0
- added joint 8_9: type revolute, parent 8, child 9, origin xyz=1.0269869044018236 0 0 rpy=0 0 0, axis 0 1 0, limit lower=-3.14159 upper=3.14159 effort=0.0 velocity=0.0
- added joint 9_10: type revolute, parent 9, child 10, origin xyz=0.8489169791059855 0 0 rpy=0 0 0, axis 0 1 0, limit lower=-3.14159 upper=3.14159 effort=0.0 velocity=0.0
- joint 0_1: axis 0 1 0 -> 0 0 1; origin xyz=0.420993414345372 0 5 rpy=0 0 0 -> xyz=0.3852877423970373 0 5 rpy=0 0 0
- joint 1_2: origin xyz=0.8382508003398526 0 0 rpy=0 0 0 -> xyz=1.176199397605837 0 0 rpy=0 0 0
- joint 2_3: axis 0 1 0 -> 0 0 1; origin xyz=1.0966477965233212 0 0 rpy=0 0 0 -> xyz=1.3958249340268583 0 0 rpy=0 0 0
- joint 3_4: origin xyz=1.1596397643018466 0 0 rpy=0 0 0 -> xyz=0.9883456458746409 0 0 rpy=0 0 0
