Commit message: Final code finished

File: horse0.urdf (robot description, URDF)
Before this commit: robot robot, 14 links, 13 joints
Links:
- removed link 10
- removed link 11
- removed link 12
- removed link 13
- removed link 7
- removed link 8
- removed link 9
- link 3: geometry collision box size=0.5248312389393546 0.46766119630913844 0.4601839010437445; visual box size=0.5248312389393546 0.46766119630913844 0.4601839010437445
- link 4: geometry collision box size=0.41516741050193706 0.35232431701892125 0.5596354831753318; visual box size=0.41516741050193706 0.35232431701892125 0.5596354831753318
- link 5: geometry collision box size=0.39982733683726157 0.3834136375514333 0.5605669163846474; visual box size=0.39982733683726157 0.3834136375514333 0.5605669163846474
- link 6: geometry collision box size=0.5145710471385195 0.3172899726724668 0.5067890606328732; visual box size=0.5145710471385195 0.3172899726724668 0.5067890606328732
Joints:
- removed joint 0_3
- removed joint 0_4
- removed joint 1_7
- removed joint 1_8
- removed joint 1_9
- removed joint 2_10
- removed joint 2_11
- removed joint 2_12
- removed joint 2_13
- added joint 1_3: type revolute, parent 1, child 3, origin xyz=0.35 0.0 0.35 rpy=0 0 0, axis 1 0 0, limit lower=-3.14159 upper=3.14159 effort=0.0 velocity=0.0
- added joint 1_4: type revolute, parent 1, child 4, origin xyz=0.0 0.0 0.4601839010437445 rpy=0 0 0, axis 0 1 0, limit lower=-3.14159 upper=3.14159 effort=0.0 velocity=0.0
- joint 1_2: axis 0 0 1 -> 0 1 0
- joint 1_5: axis 1 0 0 -> 0 1 0; origin xyz=0.35 0.35 0.0 rpy=0 0 0 -> xyz=0.0 0.0 0.5596354831753318 rpy=0 0 0
- joint 1_6: axis 0 0 1 -> 0 1 0; origin xyz=0.0 0.4673957662022229 0.0 rpy=0 0 0 -> xyz=0.0 0.0 0.5605669163846474 rpy=0 0 0

File: horse1.urdf (robot description, URDF)
Before this commit: robot robot, 9 links, 8 joints
Links:
- added link 10, mass 1; collision box size=0.6010210201211912 0.6032710029369588 0.4905108778522366; visual box size=0.6010210201211912 0.6032710029369588 0.4905108778522366
- added link 9, mass 1; collision box size=0.6941518746087403 0.7205966523683828 0.5015061266729919; visual box size=0.6941518746087403 0.7205966523683828 0.5015061266729919
- link 3: geometry collision box size=0.6761405168643262 0.504762938246162 0.35863496322006005; visual box size=0.6761405168643262 0.504762938246162 0.35863496322006005
- link 4: geometry collision box size=0.7466331472307952 0.4076487405864303 0.3793665857149137; visual box size=0.7466331472307952 0.4076487405864303 0.3793665857149137
- link 5: geometry collision box size=0.6545876429853859 0.4268376893421977 0.48392124673576714; visual box size=0.6545876429853859 0.4268376893421977 0.48392124673576714
- link 6: geometry collision box size=0.38708662969523006 0.6491001939185268 0.6570692065436203; visual box size=0.38708662969523006 0.6491001939185268 0.6570692065436203
- link 7: geometry collision box size=0.7240452109513521 0.6614423202382419 0.5075695604319685; visual box size=0.7240452109513521 0.6614423202382419 0.5075695604319685
- link 8: geometry collision box size=0.36049907664657516 0.6233157040446149 0.465768885117562; visual box size=0.36049907664657516 0.6233157040446149 0.465768885117562
Joints:
- removed joint 1_3
- removed joint 2_5
- removed joint 2_6
- removed joint 2_7
- added joint 0_3: type revolute, parent 0, child 3, origin xyz=0.0 0.0 4.625 rpy=0 0 0, axis 1 0 0, limit lower=-3.14159 upper=3.14159 effort=0.0 velocity=0.0
- added joint 1_5: type revolute, parent 1, child 5, origin xyz=0.0 -0.4076487405864303 0.0 rpy=0 0 0, axis 1 0 0, limit lower=-3.14159 upper=3.14159 effort=0.0 velocity=0.0
- added joint 1_6: type revolute, parent 1, child 6, origin xyz=0.0 -0.4268376893421977 0.0 rpy=0 0 0, axis 0 0 1, limit lower=-3.14159 upper=3.14159 effort=0.0 velocity=0.0
- added joint 1_7: type revolute, parent 1, child 7, origin xyz=0.0 -0.6491001939185268 0.0 rpy=0 0 0, axis 1 0 0, limit lower=-3.14159 upper=3.14159 effort=0.0 velocity=0.0
- added joint 2_10: type revolute, parent 2, child 10, origin xyz=0.0 0.0 -0.5015061266729919 rpy=0 0 0, axis 1 0 0, limit lower=-3.14159 upper=3.14159 effort=0.0 velocity=0.0
- added joint 2_9: type revolute, parent 2, child 9, origin xyz=0.325 0.0 -0.325 rpy=0 0 0, axis 0 1 0, limit lower=-3.14159 upper=3.14159 effort=0.0 velocity=0.0
- joint 0_1: axis 0 0 1 -> 0 1 0
- joint 1_2: axis 0 1 0 -> 0 0 1
- joint 1_4: origin xyz=0.0 -0.5576810069679553 0.0 rpy=0 0 0 -> xyz=0.35 -0.35 0.0 rpy=0 0 0
- joint 2_8: axis 1 0 0 -> 0 1 0; origin xyz=0.0 -0.6278246422232237 0.0 rpy=0 0 0 -> xyz=0.325 0.0 0.325 rpy=0 0 0

File: horse3.urdf (robot description, URDF)
Before this commit: robot robot, 9 links, 8 joints
Links:
- removed link 7
- removed link 8
- link 3: geometry collision box size=0.5248312389393546 0.46766119630913844 0.4601839010437445; visual box size=0.5248312389393546 0.46766119630913844 0.4601839010437445
- link 4: geometry collision box size=0.41516741050193706 0.35232431701892125 0.5596354831753318; visual box size=0.41516741050193706 0.35232431701892125 0.5596354831753318
- link 5: geometry collision box size=0.39982733683726157 0.3834136375514333 0.5605669163846474; visual box size=0.39982733683726157 0.3834136375514333 0.5605669163846474
- link 6: geometry collision box size=0.5145710471385195 0.3172899726724668 0.5067890606328732; visual box size=0.5145710471385195 0.3172899726724668 0.5067890606328732
Joints:
- removed joint 2_5
- removed joint 2_6
- removed joint 2_7
- removed joint 2_8
- added joint 1_5: type revolute, parent 1, child 5, origin xyz=0.0 0.0 0.5596354831753318 rpy=0 0 0, axis 0 1 0, limit lower=-3.14159 upper=3.14159 effort=0.0 velocity=0.0
- added joint 1_6: type revolute, parent 1, child 6, origin xyz=0.0 0.0 0.5605669163846474 rpy=0 0 0, axis 0 1 0, limit lower=-3.14159 upper=3.14159 effort=0.0 velocity=0.0
- joint 0_1: axis 0 0 1 -> 0 1 0
- joint 1_3: origin xyz=0.35 -0.35 0.0 rpy=0 0 0 -> xyz=0.35 0.0 0.35 rpy=0 0 0
- joint 1_4: axis 1 0 0 -> 0 1 0; origin xyz=0.0 -0.5576810069679553 0.0 rpy=0 0 0 -> xyz=0.0 0.0 0.4601839010437445 rpy=0 0 0

File: horse4.urdf (robot description, URDF)
Before this commit: robot robot, 14 links, 13 joints
Links:
- removed link 11
- removed link 12
- removed link 13
- link 10: geometry collision box size=0.6010210201211912 0.6032710029369588 0.4905108778522366; visual box size=0.6010210201211912 0.6032710029369588 0.4905108778522366
- link 3: geometry collision box size=0.6761405168643262 0.504762938246162 0.35863496322006005; visual box size=0.6761405168643262 0.504762938246162 0.35863496322006005
- link 4: geometry collision box size=0.7466331472307952 0.4076487405864303 0.3793665857149137; visual box size=0.7466331472307952 0.4076487405864303 0.3793665857149137
- link 5: geometry collision box size=0.6545876429853859 0.4268376893421977 0.48392124673576714; visual box size=0.6545876429853859 0.4268376893421977 0.48392124673576714
- link 6: geometry collision box size=0.38708662969523006 0.6491001939185268 0.6570692065436203; visual box size=0.38708662969523006 0.6491001939185268 0.6570692065436203
- link 7: geometry collision box size=0.7240452109513521 0.6614423202382419 0.5075695604319685; visual box size=0.7240452109513521 0.6614423202382419 0.5075695604319685
- link 8: geometry collision box size=0.36049907664657516 0.6233157040446149 0.465768885117562; visual box size=0.36049907664657516 0.6233157040446149 0.465768885117562
- link 9: geometry collision box size=0.6941518746087403 0.7205966523683828 0.5015061266729919; visual box size=0.6941518746087403 0.7205966523683828 0.5015061266729919
Joints:
- removed joint 0_4
- removed joint 1_8
- removed joint 1_9
- removed joint 2_11
- removed joint 2_12
- removed joint 2_13
- added joint 1_4: type revolute, parent 1, child 4, origin xyz=0.35 -0.35 0.0 rpy=0 0 0, axis 1 0 0, limit lower=-3.14159 upper=3.14159 effort=0.0 velocity=0.0
- added joint 2_8: type revolute, parent 2, child 8, origin xyz=0.325 0.0 0.325 rpy=0 0 0, axis 0 1 0, limit lower=-3.14159 upper=3.14159 effort=0.0 velocity=0.0
- added joint 2_9: type revolute, parent 2, child 9, origin xyz=0.325 0.0 -0.325 rpy=0 0 0, axis 0 1 0, limit lower=-3.14159 upper=3.14159 effort=0.0 velocity=0.0
- joint 0_3: origin xyz=0.0 0.375 5.0 rpy=0 0 0 -> xyz=0.0 0.0 4.625 rpy=0 0 0
- joint 1_5: origin xyz=0.35 0.35 0.0 rpy=0 0 0 -> xyz=0.0 -0.4076487405864303 0.0 rpy=0 0 0
- joint 1_6: origin xyz=0.0 0.4673957662022229 0.0 rpy=0 0 0 -> xyz=0.0 -0.4268376893421977 0.0 rpy=0 0 0
- joint 1_7: origin xyz=0.35 -0.35 0.0 rpy=0 0 0 -> xyz=0.0 -0.6491001939185268 0.0 rpy=0 0 0
- joint 2_10: axis 0 1 0 -> 1 0 0; origin xyz=0.325 0.0 0.325 rpy=0 0 0 -> xyz=0.0 0.0 -0.5015061266729919 rpy=0 0 0

File: horse5.urdf (robot description, URDF)
Before this commit: robot robot, 9 links, 8 joints
Links:
- removed link 7
- removed link 8
- link 3: geometry collision box size=0.2951851861309304 0.4291201546607567 0.2594925637112075; visual box size=0.2951851861309304 0.4291201546607567 0.2594925637112075
- link 4: geometry collision box size=0.47501336111883485 0.26518412633339483 0.38517698434140196; visual box size=0.47501336111883485 0.26518412633339483 0.38517698434140196
- link 5: geometry collision box size=0.25129128850862925 0.46687295768568937 0.5435871020527727; visual box size=0.25129128850862925 0.46687295768568937 0.5435871020527727
- link 6: geometry collision box size=0.7459921276333181 0.4677604118288111 0.4312136888766655; visual box size=0.7459921276333181 0.4677604118288111 0.4312136888766655
Joints:
- removed joint 1_3
- removed joint 1_4
- removed joint 2_5
- removed joint 2_6
- removed joint 2_7
- removed joint 2_8
- added joint 0_3: type revolute, parent 0, child 3, origin xyz=0.0 0.0 4.625 rpy=0 0 0, axis 0 1 0, limit lower=-3.14159 upper=3.14159 effort=0.0 velocity=0.0
- added joint 0_4: type revolute, parent 0, child 4, origin xyz=0.0 0.0 -0.2594925637112075 rpy=0 0 0, axis 1 0 0, limit lower=-3.14159 upper=3.14159 effort=0.0 velocity=0.0
- added joint 0_5: type revolute, parent 0, child 5, origin xyz=0.0 0.0 -0.38517698434140196 rpy=0 0 0, axis 0 1 0, limit lower=-3.14159 upper=3.14159 effort=0.0 velocity=0.0
- added joint 0_6: type revolute, parent 0, child 6, origin xyz=0.0 0.0 -0.5435871020527727 rpy=0 0 0, axis 1 0 0, limit lower=-3.14159 upper=3.14159 effort=0.0 velocity=0.0
- joint 1_2: axis 0 1 0 -> 0 0 1
