Commit message: Trying to fix joint intersections

File: horse.urdf (robot description, URDF)
Before this commit: robot robot, 10 links, 9 joints
Links:
- added link 10, mass 1; collision box size=0.2683388061049887 0.32039339119817095 0.5175249294992867; visual box size=0.2683388061049887 0.32039339119817095 0.5175249294992867
- added link 11, mass 1; collision box size=0.6164368964805801 0.7242635065451741 0.32676584558895977; visual box size=0.6164368964805801 0.7242635065451741 0.32676584558895977
- added link 12, mass 1; collision box size=0.5744521487274462 0.5799148729258465 0.5081728397356853; visual box size=0.5744521487274462 0.5799148729258465 0.5081728397356853
- added link 13, mass 1; collision box size=0.53614415538739 0.53318255080987 0.6234742544872398; visual box size=0.53614415538739 0.53318255080987 0.6234742544872398
- link 0: geometry collision box size=0.7105355723470106 0.44830577543271816 0.7117931167454707; visual box size=0.7105355723470106 0.44830577543271816 0.7117931167454707
- link 1: geometry collision box size=0.7194816190780835 0.36364739526863293 0.3230331040053642; visual box size=0.7194816190780835 0.36364739526863293 0.3230331040053642
- link 2: geometry collision box size=0.7143647897648868 0.5325170877214125 0.28154931324767823; visual box size=0.7143647897648868 0.5325170877214125 0.28154931324767823
- link 3: geometry collision box size=0.6780817988938268 0.7015674529970847 0.4159924379321928; visual box size=0.6780817988938268 0.7015674529970847 0.4159924379321928
- link 4: geometry collision box size=0.3366908237145363 0.6946865018724873 0.6584952133944284; visual box size=0.3366908237145363 0.6946865018724873 0.6584952133944284
- link 5: geometry collision box size=0.6748811363100236 0.6445975853585777 0.7237183180664166; visual box size=0.6748811363100236 0.6445975853585777 0.7237183180664166
- link 6: geometry collision box size=0.5052836175469078 0.40663261822158747 0.519916468723904; visual box size=0.5052836175469078 0.40663261822158747 0.519916468723904
- link 7: geometry collision box size=0.44388462139812274 0.2967907488510801 0.5854102537332929; visual box size=0.44388462139812274 0.2967907488510801 0.5854102537332929
- link 8: geometry collision box size=0.7455417670586415 0.2599277787387809 0.40495467332904983; visual box size=0.7455417670586415 0.2599277787387809 0.40495467332904983
- link 9: geometry collision box size=0.5210399546502268 0.3418600731738085 0.41335436366812667; visual box size=0.5210399546502268 0.3418600731738085 0.41335436366812667
Joints:
- added joint 10_11: type revolute, parent 10, child 11, origin xyz=0.2683388061049887 0.0 0.5175249294992867 rpy=0 0 0, axis 0 1 0, limit lower=-3.14159 upper=3.14159 effort=0.0 velocity=0.0
- added joint 11_12: type revolute, parent 11, child 12, origin xyz=0.6164368964805801 0.0 0.32676584558895977 rpy=0 0 0, axis 1 0 0, limit lower=-3.14159 upper=3.14159 effort=0.0 velocity=0.0
- added joint 12_13: type revolute, parent 12, child 13, origin xyz=0.0 0.5799148729258465 0.5081728397356853 rpy=0 0 0, axis 0 0 1, limit lower=-3.14159 upper=3.14159 effort=0.0 velocity=0.0
- added joint 9_10: type revolute, parent 9, child 10, origin xyz=0.5210399546502268 0.0 0.41335436366812667 rpy=0 0 0, axis 0 1 0, limit lower=-3.14159 upper=3.14159 effort=0.0 velocity=0.0
- joint 0_1: axis 0 0 1 -> 1 0 0; origin xyz=0.19634867832014513 0.0 5.0 rpy=0 0 0 -> xyz=0.0 0.22415288771635908 0.35589655837273537 rpy=0 0 0
- joint 1_2: axis 0 1 0 -> 1 0 0; origin xyz=0.6510393307305515 0.0 0.0 rpy=0 0 0 -> xyz=0.0 0.0 0.6460662080107284 rpy=0 0 0
- joint 2_3: axis 0 1 0 -> 1 0 0; origin xyz=0.459289111520379 0.0 0.0 rpy=0 0 0 -> xyz=0.0 0.0 0.5630986264953565 rpy=0 0 0
- joint 3_4: axis 0 0 1 -> 1 0 0; origin xyz=0.46910464358221565 0.0 0.0 rpy=0 0 0 -> xyz=0.0 0.7015674529970847 0.4159924379321928 rpy=0 0 0
- joint 4_5: axis 0 1 0 -> 0 0 1; origin xyz=0.6474035050006905 0.0 0.0 rpy=0 0 0 -> xyz=0.3366908237145363 0.6946865018724873 0.0 rpy=0 0 0
- joint 5_6: axis 0 0 1 -> 0 1 0; origin xyz=0.0 0.6039017505143294 0.0 rpy=0 0 0 -> xyz=0.6748811363100236 0.0 0.7237183180664166 rpy=0 0 0
- joint 6_7: origin xyz=0.0 0.26116666050769477 0.0 rpy=0 0 0 -> xyz=0.5052836175469078 0.0 0.519916468723904 rpy=0 0 0
- joint 7_8: axis 0 1 0 -> 1 0 0; origin xyz=0.0 0.0 0.2709632013636881 rpy=0 0 0 -> xyz=0.44388462139812274 0.0 0.5854102537332929 rpy=0 0 0
- joint 8_9: origin xyz=0.0 0.5821213068929524 0.0 rpy=0 0 0 -> xyz=0.7455417670586415 0.0 0.40495467332904983 rpy=0 0 0

Commit message: Fixed joint intersections

File: horse.urdf (robot description, URDF)
Before this commit: robot robot, 14 links, 13 joints
Links:
- removed link 10
- removed link 11
- removed link 12
- removed link 13
- link 0: geometry collision box size=0.3555374812396278 0.5968131718329033 0.5119662864539396; visual box size=0.3555374812396278 0.5968131718329033 0.5119662864539396
- link 1: geometry collision box size=0.44885612324530777 0.27214384509317674 0.5599144589873505; visual box size=0.44885612324530777 0.27214384509317674 0.5599144589873505
- link 2: geometry collision box size=0.46534219470182075 0.360891065933566 0.38075246492314263; visual box size=0.46534219470182075 0.360891065933566 0.38075246492314263
- link 3: geometry collision box size=0.27138387687509496 0.7047381906713365 0.4421425654242621; visual box size=0.27138387687509496 0.7047381906713365 0.4421425654242621
- link 4: geometry collision box size=0.48167571362975675 0.36888922497869836 0.7266033631900408; visual box size=0.48167571362975675 0.36888922497869836 0.7266033631900408
- link 5: geometry collision box size=0.7456622376039774 0.6684323222281978 0.6151780407809158; visual box size=0.7456622376039774 0.6684323222281978 0.6151780407809158
- link 6: geometry collision box size=0.3882099247784682 0.5981350490973 0.7164651185520443; visual box size=0.3882099247784682 0.5981350490973 0.7164651185520443
- link 7: geometry collision box size=0.7100771290993935 0.5973501301876555 0.42312335831890285; visual box size=0.7100771290993935 0.5973501301876555 0.42312335831890285
- link 8: geometry collision box size=0.3525208727965242 0.26321247934202596 0.45520925116756833; visual box size=0.3525208727965242 0.26321247934202596 0.45520925116756833
- link 9: geometry collision box size=0.55039466261764 0.5295920191789012 0.5717871138862461; visual box size=0.55039466261764 0.5295920191789012 0.5717871138862461
Joints:
- removed joint 10_11
- removed joint 11_12
- removed joint 12_13
- removed joint 9_10
- joint 0_1: axis 1 0 0 -> 0 1 0; origin xyz=0.0 0.22415288771635908 0.35589655837273537 rpy=0 0 0 -> xyz=0.1777687406198139 0.0 0.0 rpy=0 0 0
- joint 1_2: axis 1 0 0 -> 0 0 1; origin xyz=0.0 0.0 0.6460662080107284 rpy=0 0 0 -> xyz=0.44885612324530777 0.0 0.0 rpy=0 0 0
- joint 2_3: axis 1 0 0 -> 0 0 1; origin xyz=0.0 0.0 0.5630986264953565 rpy=0 0 0 -> xyz=0.23267109735091038 0.180445532966783 0.0 rpy=0 0 0
- joint 3_4: axis 1 0 0 -> 0 0 1; origin xyz=0.0 0.7015674529970847 0.4159924379321928 rpy=0 0 0 -> xyz=0.0 0.7047381906713365 0.0 rpy=0 0 0
- joint 4_5: origin xyz=0.3366908237145363 0.6946865018724873 0.0 rpy=0 0 0 -> xyz=0.24083785681487838 0.18444461248934918 0.0 rpy=0 0 0
- joint 5_6: origin xyz=0.6748811363100236 0.0 0.7237183180664166 rpy=0 0 0 -> xyz=0.7456622376039774 0.0 0.0 rpy=0 0 0
- joint 6_7: origin xyz=0.5052836175469078 0.0 0.519916468723904 rpy=0 0 0 -> xyz=0.3882099247784682 0.0 0.0 rpy=0 0 0
- joint 7_8: axis 1 0 0 -> 0 0 1; origin xyz=0.44388462139812274 0.0 0.5854102537332929 rpy=0 0 0 -> xyz=0.7100771290993935 0.0 0.0 rpy=0 0 0
- joint 8_9: axis 0 0 1 -> 1 0 0; origin xyz=0.7455417670586415 0.0 0.40495467332904983 rpy=0 0 0 -> xyz=0.1762604363982621 0.0 0.22760462558378416 rpy=0 0 0

Commit message: Commit

File: horse.urdf (robot description, URDF)
Before this commit: robot robot, 10 links, 9 joints
Links:
- added link 10, mass 1; collision box size=0.5395244143293867 0.32804260791308626 0.25372033572988606; visual box size=0.5395244143293867 0.32804260791308626 0.25372033572988606
- added link 11, mass 1; collision box size=0.5321439578707785 0.637051817614301 0.6294899656250453; visual box size=0.5321439578707785 0.637051817614301 0.6294899656250453
- added link 12, mass 1; collision box size=0.6472652640651526 0.47799698910171107 0.46603442032711645; visual box size=0.6472652640651526 0.47799698910171107 0.46603442032711645
- added link 13, mass 1; collision box size=0.5610815900408204 0.6675424416328586 0.35467195645228133; visual box size=0.5610815900408204 0.6675424416328586 0.35467195645228133
- added link 14, mass 1; collision box size=0.4965035350427981 0.37021541064423147 0.6870023178009423; visual box size=0.4965035350427981 0.37021541064423147 0.6870023178009423
- link 0: geometry collision box size=0.5390104152002784 0.7453039405006765 0.30433523762044024; visual box size=0.5390104152002784 0.7453039405006765 0.30433523762044024
- link 1: geometry collision box size=0.4729137931943257 0.7308397207012318 0.41981447219636553; visual box size=0.4729137931943257 0.7308397207012318 0.41981447219636553
- link 2: geometry collision box size=0.5389488494277829 0.296941890291935 0.4677023037709393; visual box size=0.5389488494277829 0.296941890291935 0.4677023037709393
- link 3: geometry collision box size=0.4558319382378959 0.7304713686608535 0.3403958616028942; visual box size=0.4558319382378959 0.7304713686608535 0.3403958616028942
- link 4: geometry collision box size=0.48238450993940946 0.27856228788420884 0.3119849430614323; visual box size=0.48238450993940946 0.27856228788420884 0.3119849430614323
- link 5: geometry collision box size=0.3758302596269274 0.4786762545239609 0.5961949027229265; visual box size=0.3758302596269274 0.4786762545239609 0.5961949027229265
- link 6: geometry collision box size=0.3115930538218966 0.4835471362875196 0.4859856884534575; visual box size=0.3115930538218966 0.4835471362875196 0.4859856884534575
- link 7: geometry collision box size=0.4162883875689276 0.2932560412197484 0.2891236109674334; visual box size=0.4162883875689276 0.2932560412197484 0.2891236109674334
- link 8: geometry collision box size=0.3141446143462831 0.34404426440432934 0.5283045860204525; visual box size=0.3141446143462831 0.34404426440432934 0.5283045860204525
- link 9: geometry collision box size=0.6640400814900527 0.42160065738763186 0.6018734228399392; visual box size=0.6640400814900527 0.42160065738763186 0.6018734228399392
Joints:
- added joint 10_11: type revolute, parent 10, child 11, origin xyz=0.26976220716469335 0.16402130395654313 0.0 rpy=0 0 0, axis 0 1 0, limit lower=-3.14159 upper=3.14159 effort=0.0 velocity=0.0
- added joint 11_12: type revolute, parent 11, child 12, origin xyz=0.26607197893538925 0.3185259088071505 0.0 rpy=0 0 0, axis 1 0 0, limit lower=-3.14159 upper=3.14159 effort=0.0 velocity=0.0
- added joint 12_13: type revolute, parent 12, child 13, origin xyz=0.3236326320325763 0.23899849455085553 0.0 rpy=0 0 0, axis 0 0 1, limit lower=-3.14159 upper=3.14159 effort=0.0 velocity=0.0
- added joint 13_14: type revolute, parent 13, child 14, origin xyz=0.5610815900408204 0.0 0.0 rpy=0 0 0, axis 0 1 0, limit lower=-3.14159 upper=3.14159 effort=0.0 velocity=0.0
- added joint 9_10: type revolute, parent 9, child 10, origin xyz=0.0 0.21080032869381593 0.3009367114199696 rpy=0 0 0, axis 0 0 1, limit lower=-3.14159 upper=3.14159 effort=0.0 velocity=0.0
- joint 0_1: origin xyz=0.1777687406198139 0.0 0.0 rpy=0 0 0 -> xyz=0.0 0.0 0.15216761881022012 rpy=0 0 0
- joint 1_2: axis 0 0 1 -> 0 1 0; origin xyz=0.44885612324530777 0.0 0.0 rpy=0 0 0 -> xyz=0.0 0.0 0.41981447219636553 rpy=0 0 0
- joint 2_3: axis 0 0 1 -> 1 0 0; origin xyz=0.23267109735091038 0.180445532966783 0.0 rpy=0 0 0 -> xyz=0.0 0.0 0.4677023037709393 rpy=0 0 0
- joint 3_4: axis 0 0 1 -> 0 1 0; origin xyz=0.0 0.7047381906713365 0.0 rpy=0 0 0 -> xyz=0.22791596911894796 0.0 0.1701979308014471 rpy=0 0 0
- joint 4_5: axis 0 0 1 -> 0 1 0; origin xyz=0.24083785681487838 0.18444461248934918 0.0 rpy=0 0 0 -> xyz=0.48238450993940946 0.0 0.0 rpy=0 0 0
- joint 5_6: axis 0 1 0 -> 0 0 1; origin xyz=0.7456622376039774 0.0 0.0 rpy=0 0 0 -> xyz=0.1879151298134637 0.23933812726198045 0.0 rpy=0 0 0
- joint 6_7: axis 0 1 0 -> 1 0 0; origin xyz=0.3882099247784682 0.0 0.0 rpy=0 0 0 -> xyz=0.0 0.4835471362875196 0.0 rpy=0 0 0
- joint 7_8: axis 0 0 1 -> 0 1 0; origin xyz=0.7100771290993935 0.0 0.0 rpy=0 0 0 -> xyz=0.2081441937844638 0.1466280206098742 0.0 rpy=0 0 0
- joint 8_9: axis 1 0 0 -> 0 1 0; origin xyz=0.1762604363982621 0.0 0.22760462558378416 rpy=0 0 0 -> xyz=0.15707230717314155 0.0 0.26415229301022625 rpy=0 0 0
