Commit message: Self-collisions need fixing, otherwise all done
There is some bug in horseInfo.Construct_Limb() which is causing the bodies to form joints within each other. I have been debugging for 4 hours and can't find the issue. Need to check this out later.

File: horse.urdf (robot description, URDF)
Before this commit: robot robot, 15 links, 14 joints
Links:
- added link 15, mass 1; collision box size=0.6024526312017453 0.7174931611696186 0.31115111834961096; visual box size=0.6024526312017453 0.7174931611696186 0.31115111834961096
- added link 16, mass 1; collision box size=0.2660885050224523 0.727725250204692 0.2965071215549385; visual box size=0.2660885050224523 0.727725250204692 0.2965071215549385
- added link 17, mass 1; collision box size=0.4155040237337591 0.3569332577138792 0.6400870679768936; visual box size=0.4155040237337591 0.3569332577138792 0.6400870679768936
- added link 18, mass 1; collision box size=0.41702055193325355 0.436069531312529 0.46152882576014037; visual box size=0.41702055193325355 0.436069531312529 0.46152882576014037
- added link 19, mass 1; collision box size=0.34809326373159366 0.602911158098119 0.3043780492221309; visual box size=0.34809326373159366 0.602911158098119 0.3043780492221309
- added link 20, mass 1; collision box size=0.7242457683387034 0.5447396700238806 0.42053057262424975; visual box size=0.7242457683387034 0.5447396700238806 0.42053057262424975
- added link 21, mass 1; collision box size=0.5844564189771404 0.7409299422342122 0.7214121691888015; visual box size=0.5844564189771404 0.7409299422342122 0.7214121691888015
- added link 22, mass 1; collision box size=0.30308672549643095 0.360977274473781 0.6584474884297566; visual box size=0.30308672549643095 0.360977274473781 0.6584474884297566
- added link 23, mass 1; collision box size=0.6308687781669662 0.3965356615486386 0.602664197459892; visual box size=0.6308687781669662 0.3965356615486386 0.602664197459892
- added link 24, mass 1; collision box size=0.3708266042462652 0.5342649234255765 0.5205221972466842; visual box size=0.3708266042462652 0.5342649234255765 0.5205221972466842
- added link 25, mass 1; collision box size=0.5547939837906293 0.7079581160455666 0.501482182370823; visual box size=0.5547939837906293 0.7079581160455666 0.501482182370823
- added link 26, mass 1; collision box size=0.6918299757108495 0.6052051336667426 0.4300479260882413; visual box size=0.6918299757108495 0.6052051336667426 0.4300479260882413
- added link 27, mass 1; collision box size=0.45749206256191893 0.6560939371181862 0.5126138453347886; visual box size=0.45749206256191893 0.6560939371181862 0.5126138453347886
- added link 28, mass 1; collision box size=0.6159124446848796 0.6303935875980469 0.2913912834376072; visual box size=0.6159124446848796 0.6303935875980469 0.2913912834376072
- added link 29, mass 1; collision box size=0.6055017866194479 0.4232720186454721 0.6367859776100915; visual box size=0.6055017866194479 0.4232720186454721 0.6367859776100915
- added link 30, mass 1; collision box size=0.6688022428902598 0.7125338294204874 0.6962245388298368; visual box size=0.6688022428902598 0.7125338294204874 0.6962245388298368
- added link 31, mass 1; collision box size=0.7443212092358178 0.7326944040478536 0.3516152457727334; visual box size=0.7443212092358178 0.7326944040478536 0.3516152457727334
- added link 32, mass 1; collision box size=0.4624481338874678 0.6252786007918256 0.2772820687882443; visual box size=0.4624481338874678 0.6252786007918256 0.2772820687882443
- added link 33, mass 1; collision box size=0.5439791401394525 0.45611777589360186 0.4312691904410735; visual box size=0.5439791401394525 0.45611777589360186 0.4312691904410735
- added link 34, mass 1; collision box size=0.2623105684578354 0.28149671068957277 0.49636744322829557; visual box size=0.2623105684578354 0.28149671068957277 0.49636744322829557
- added link 35, mass 1; collision box size=0.4537037372078289 0.7153420178226213 0.30124879931176074; visual box size=0.4537037372078289 0.7153420178226213 0.30124879931176074
- added link 36, mass 1; collision box size=0.31677454028423957 0.5907710163848692 0.5530395556316873; visual box size=0.31677454028423957 0.5907710163848692 0.5530395556316873
- added link 37, mass 1; collision box size=0.4696746226306808 0.2888790144587677 0.3976821399185429; visual box size=0.4696746226306808 0.2888790144587677 0.3976821399185429
- added link 38, mass 1; collision box size=0.7233742842884578 0.2688797049139123 0.7127452342019391; visual box size=0.7233742842884578 0.2688797049139123 0.7127452342019391
- added link 39, mass 1; collision box size=0.5854065644112496 0.6584559039213599 0.6234129349109545; visual box size=0.5854065644112496 0.6584559039213599 0.6234129349109545
- added link 40, mass 1; collision box size=0.3556535125824758 0.729892256556159 0.4729350153164811; visual box size=0.3556535125824758 0.729892256556159 0.4729350153164811
- added link 41, mass 1; collision box size=0.28498712145338395 0.4872400253486729 0.3649910883309176; visual box size=0.28498712145338395 0.4872400253486729 0.3649910883309176
- added link 42, mass 1; collision box size=0.31548826332740254 0.7286006727177956 0.36080082242057093; visual box size=0.31548826332740254 0.7286006727177956 0.36080082242057093
- added link 43, mass 1; collision box size=0.6724398201588286 0.49284939497623753 0.4074692052581001; visual box size=0.6724398201588286 0.49284939497623753 0.4074692052581001
- added link 44, mass 1; collision box size=0.39067342588903525 0.4288362886365232 0.6392121403820734; visual box size=0.39067342588903525 0.4288362886365232 0.6392121403820734
- added link 45, mass 1; collision box size=0.5948266489659901 0.37645777652859197 0.380988574375948; visual box size=0.5948266489659901 0.37645777652859197 0.380988574375948
- added link 46, mass 1; collision box size=0.6041985786675705 0.48532097082509085 0.6704571751124948; visual box size=0.6041985786675705 0.48532097082509085 0.6704571751124948
- added link 47, mass 1; collision box size=0.2673174848600397 0.43431165844059466 0.3783782410105099; visual box size=0.2673174848600397 0.43431165844059466 0.3783782410105099
- added link 48, mass 1; collision box size=0.5874113202432064 0.5682766222081965 0.4355230788582382; visual box size=0.5874113202432064 0.5682766222081965 0.4355230788582382
- added link 49, mass 1; collision box size=0.6627807888888702 0.539477252072275 0.6042971082613806; visual box size=0.6627807888888702 0.539477252072275 0.6042971082613806
- added link 50, mass 1; collision box size=0.7227320940855906 0.6949054448825084 0.3603917300681739; visual box size=0.7227320940855906 0.6949054448825084 0.3603917300681739
- added link 51, mass 1; collision box size=0.47497344128809404 0.43310370187053904 0.479037828185724; visual box size=0.47497344128809404 0.43310370187053904 0.479037828185724
- added link 52, mass 1; collision box size=0.5305084518739983 0.4431953411787529 0.6939525223000419; visual box size=0.5305084518739983 0.4431953411787529 0.6939525223000419
- added link 53, mass 1; collision box size=0.3314795504042853 0.7418884764454653 0.7226840859919716; visual box size=0.3314795504042853 0.7418884764454653 0.7226840859919716
- added link 54, mass 1; collision box size=0.34313659021996956 0.3654371131979153 0.4940660578440078; visual box size=0.34313659021996956 0.3654371131979153 0.4940660578440078
- link 0: geometry collision box size=0.49897261603943965 0.3956758299960858 0.3567633440639782; visual box size=0.49897261603943965 0.3956758299960858 0.3567633440639782
- link 1: geometry collision box size=0.5846085752986323 0.3745064011564245 0.7426855955938925; visual box size=0.5846085752986323 0.3745064011564245 0.7426855955938925
- link 10: geometry collision box size=0.7159926239791925 0.2501426365879886 0.2767726126793666; visual box size=0.7159926239791925 0.2501426365879886 0.2767726126793666
- link 11: geometry collision box size=0.31787989455068444 0.520496103101418 0.3738625065206649; visual box size=0.31787989455068444 0.520496103101418 0.3738625065206649
- link 12: geometry collision box size=0.4413054327103169 0.5884093426108693 0.2699834825965733; visual box size=0.4413054327103169 0.5884093426108693 0.2699834825965733
- link 13: geometry collision box size=0.26133968982396616 0.4376478813097882 0.3819553186343993; visual box size=0.26133968982396616 0.4376478813097882 0.3819553186343993
- link 14: geometry collision box size=0.38035754322418475 0.7398299147996006 0.5107967656374386; visual box size=0.38035754322418475 0.7398299147996006 0.5107967656374386
- link 2: geometry collision box size=0.7433821682980615 0.5487095567140214 0.635712248042587; visual box size=0.7433821682980615 0.5487095567140214 0.635712248042587
- link 3: geometry collision box size=0.5748492174148299 0.4015055511376921 0.32499027996984187; visual box size=0.5748492174148299 0.4015055511376921 0.32499027996984187
- link 4: geometry collision box size=0.30712518384142645 0.7308539585711095 0.7486950553480036; visual box size=0.30712518384142645 0.7308539585711095 0.7486950553480036
- link 5: geometry collision box size=0.31573843577023614 0.4556929607867905 0.5573973122003166; visual box size=0.31573843577023614 0.4556929607867905 0.5573973122003166
- link 6: geometry collision box size=0.3680213149510034 0.31509732215680475 0.45493899351982464; visual box size=0.3680213149510034 0.31509732215680475 0.45493899351982464
- link 7: geometry collision box size=0.6813475850688819 0.7373642221112688 0.49754032766927053; visual box size=0.6813475850688819 0.7373642221112688 0.49754032766927053
- link 8: geometry collision box size=0.7055565832717257 0.5900883511200627 0.28825234844415676; visual box size=0.7055565832717257 0.5900883511200627 0.28825234844415676
- link 9: geometry collision box size=0.6809120636500556 0.39867728068175307 0.3935170690987244; visual box size=0.6809120636500556 0.39867728068175307 0.3935170690987244
Joints:
- removed joint 11_12
- removed joint 12_13
- removed joint 13_14
- added joint 10_52: type revolute, parent 10, child 52, origin xyz=-0.35799631198959625 -0.1250713182939943 0.0 rpy=0 0 0, axis 0 0 1, limit lower=-3.14159 upper=3.14159 effort=0.0 velocity=0.0
- added joint 10_53: type revolute, parent 10, child 53, origin xyz=-0.5305084518739983 0.0 0.0 rpy=0 0 0, axis 0 0 1, limit lower=-3.14159 upper=3.14159 effort=0.0 velocity=0.0
- added joint 10_54: type revolute, parent 10, child 54, origin xyz=-0.3314795504042853 0.0 0.0 rpy=0 0 0, axis 0 1 0, limit lower=-3.14159 upper=3.14159 effort=0.0 velocity=0.0
- added joint 2_12: type revolute, parent 2, child 12, origin xyz=0.0 -0.2743547783570107 0.3178561240212935 rpy=0 0 0, axis 1 0 0, limit lower=-3.14159 upper=3.14159 effort=0.0 velocity=0.0
- added joint 2_13: type revolute, parent 2, child 13, origin xyz=0.0 0.0 0.2699834825965733 rpy=0 0 0, axis 1 0 0, limit lower=-3.14159 upper=3.14159 effort=0.0 velocity=0.0
- added joint 2_14: type revolute, parent 2, child 14, origin xyz=0.0 0.0 0.3819553186343993 rpy=0 0 0, axis 0 1 0, limit lower=-3.14159 upper=3.14159 effort=0.0 velocity=0.0
- added joint 2_15: type revolute, parent 2, child 15, origin xyz=0.0 0.0 0.5107967656374386 rpy=0 0 0, axis 1 0 0, limit lower=-3.14159 upper=3.14159 effort=0.0 velocity=0.0
- added joint 2_16: type revolute, parent 2, child 16, origin xyz=0.0 0.0 0.31115111834961096 rpy=0 0 0, axis 1 0 0, limit lower=-3.14159 upper=3.14159 effort=0.0 velocity=0.0
- added joint 4_17: type revolute, parent 4, child 17, origin xyz=0.0 -0.36542697928555473 0.3743475276740018 rpy=0 0 0, axis 0 1 0, limit lower=-3.14159 upper=3.14159 effort=0.0 velocity=0.0
- added joint 4_18: type revolute, parent 4, child 18, origin xyz=0.0 0.0 0.6400870679768936 rpy=0 0 0, axis 1 0 0, limit lower=-3.14159 upper=3.14159 effort=0.0 velocity=0.0
- added joint 4_19: type revolute, parent 4, child 19, origin xyz=0.0 -0.36542697928555473 -0.3743475276740018 rpy=0 0 0, axis 0 1 0, limit lower=-3.14159 upper=3.14159 effort=0.0 velocity=0.0
- added joint 4_20: type revolute, parent 4, child 20, origin xyz=0.0 0.0 -0.3043780492221309 rpy=0 0 0, axis 1 0 0, limit lower=-3.14159 upper=3.14159 effort=0.0 velocity=0.0
- added joint 5_21: type revolute, parent 5, child 21, origin xyz=0.15786921788511807 -0.22784648039339525 0.0 rpy=0 0 0, axis 0 1 0, limit lower=-3.14159 upper=3.14159 effort=0.0 velocity=0.0
- added joint 5_22: type revolute, parent 5, child 22, origin xyz=0.5844564189771404 0.0 0.0 rpy=0 0 0, axis 0 0 1, limit lower=-3.14159 upper=3.14159 effort=0.0 velocity=0.0
- added joint 5_23: type revolute, parent 5, child 23, origin xyz=0.30308672549643095 0.0 0.0 rpy=0 0 0, axis 0 1 0, limit lower=-3.14159 upper=3.14159 effort=0.0 velocity=0.0
- added joint 5_24: type revolute, parent 5, child 24, origin xyz=-0.15786921788511807 -0.22784648039339525 0.0 rpy=0 0 0, axis 0 1 0, limit lower=-3.14159 upper=3.14159 effort=0.0 velocity=0.0
- added joint 5_25: type revolute, parent 5, child 25, origin xyz=-0.3708266042462652 0.0 0.0 rpy=0 0 0, axis 0 1 0, limit lower=-3.14159 upper=3.14159 effort=0.0 velocity=0.0
- added joint 5_26: type revolute, parent 5, child 26, origin xyz=-0.5547939837906293 0.0 0.0 rpy=0 0 0, axis 0 0 1, limit lower=-3.14159 upper=3.14159 effort=0.0 velocity=0.0
- added joint 5_27: type revolute, parent 5, child 27, origin xyz=-0.6918299757108495 0.0 0.0 rpy=0 0 0, axis 0 0 1, limit lower=-3.14159 upper=3.14159 effort=0.0 velocity=0.0
- added joint 6_28: type revolute, parent 6, child 28, origin xyz=0.1840106574755017 -0.15754866107840237 0.0 rpy=0 0 0, axis 0 1 0, limit lower=-3.14159 upper=3.14159 effort=0.0 velocity=0.0
- added joint 6_29: type revolute, parent 6, child 29, origin xyz=0.6159124446848796 0.0 0.0 rpy=0 0 0, axis 0 0 1, limit lower=-3.14159 upper=3.14159 effort=0.0 velocity=0.0
- added joint 6_30: type revolute, parent 6, child 30, origin xyz=0.6055017866194479 0.0 0.0 rpy=0 0 0, axis 0 0 1, limit lower=-3.14159 upper=3.14159 effort=0.0 velocity=0.0
- added joint 6_31: type revolute, parent 6, child 31, origin xyz=0.6688022428902598 0.0 0.0 rpy=0 0 0, axis 0 1 0, limit lower=-3.14159 upper=3.14159 effort=0.0 velocity=0.0
- added joint 6_32: type revolute, parent 6, child 32, origin xyz=0.7443212092358178 0.0 0.0 rpy=0 0 0, axis 0 0 1, limit lower=-3.14159 upper=3.14159 effort=0.0 velocity=0.0
- added joint 7_33: type revolute, parent 7, child 33, origin xyz=0.34067379253444097 -0.3686821110556344 0.0 rpy=0 0 0, axis 0 1 0, limit lower=-3.14159 upper=3.14159 effort=0.0 velocity=0.0
- added joint 7_34: type revolute, parent 7, child 34, origin xyz=0.5439791401394525 0.0 0.0 rpy=0 0 0, axis 0 1 0, limit lower=-3.14159 upper=3.14159 effort=0.0 velocity=0.0
- added joint 7_35: type revolute, parent 7, child 35, origin xyz=0.2623105684578354 0.0 0.0 rpy=0 0 0, axis 0 1 0, limit lower=-3.14159 upper=3.14159 effort=0.0 velocity=0.0
- added joint 7_36: type revolute, parent 7, child 36, origin xyz=0.4537037372078289 0.0 0.0 rpy=0 0 0, axis 0 0 1, limit lower=-3.14159 upper=3.14159 effort=0.0 velocity=0.0
- added joint 7_37: type revolute, parent 7, child 37, origin xyz=0.31677454028423957 0.0 0.0 rpy=0 0 0, axis 0 1 0, limit lower=-3.14159 upper=3.14159 effort=0.0 velocity=0.0
- added joint 8_38: type revolute, parent 8, child 38, origin xyz=0.0 -0.2950441755600314 0.14412617422207838 rpy=0 0 0, axis 1 0 0, limit lower=-3.14159 upper=3.14159 effort=0.0 velocity=0.0
- added joint 8_39: type revolute, parent 8, child 39, origin xyz=0.0 0.0 0.7127452342019391 rpy=0 0 0, axis 1 0 0, limit lower=-3.14159 upper=3.14159 effort=0.0 velocity=0.0
- added joint 8_40: type revolute, parent 8, child 40, origin xyz=0.0 0.0 0.6234129349109545 rpy=0 0 0, axis 0 1 0, limit lower=-3.14159 upper=3.14159 effort=0.0 velocity=0.0
- added joint 8_41: type revolute, parent 8, child 41, origin xyz=0.0 0.0 0.4729350153164811 rpy=0 0 0, axis 1 0 0, limit lower=-3.14159 upper=3.14159 effort=0.0 velocity=0.0
- added joint 8_42: type revolute, parent 8, child 42, origin xyz=0.0 0.0 0.3649910883309176 rpy=0 0 0, axis 1 0 0, limit lower=-3.14159 upper=3.14159 effort=0.0 velocity=0.0
- added joint 8_43: type revolute, parent 8, child 43, origin xyz=0.0 -0.2950441755600314 -0.14412617422207838 rpy=0 0 0, axis 1 0 0, limit lower=-3.14159 upper=3.14159 effort=0.0 velocity=0.0
- added joint 8_44: type revolute, parent 8, child 44, origin xyz=0.0 0.0 -0.4074692052581001 rpy=0 0 0, axis 0 1 0, limit lower=-3.14159 upper=3.14159 effort=0.0 velocity=0.0
- added joint 9_45: type revolute, parent 9, child 45, origin xyz=0.0 -0.19933864034087653 0.1967585345493622 rpy=0 0 0, axis 0 1 0, limit lower=-3.14159 upper=3.14159 effort=0.0 velocity=0.0
- added joint 9_46: type revolute, parent 9, child 46, origin xyz=0.0 0.0 0.380988574375948 rpy=0 0 0, axis 1 0 0, limit lower=-3.14159 upper=3.14159 effort=0.0 velocity=0.0
- added joint 9_47: type revolute, parent 9, child 47, origin xyz=0.0 0.0 0.6704571751124948 rpy=0 0 0, axis 1 0 0, limit lower=-3.14159 upper=3.14159 effort=0.0 velocity=0.0
- added joint 9_48: type revolute, parent 9, child 48, origin xyz=0.0 0.0 0.3783782410105099 rpy=0 0 0, axis 0 1 0, limit lower=-3.14159 upper=3.14159 effort=0.0 velocity=0.0
- added joint 9_49: type revolute, parent 9, child 49, origin xyz=0.0 0.0 0.4355230788582382 rpy=0 0 0, axis 1 0 0, limit lower=-3.14159 upper=3.14159 effort=0.0 velocity=0.0
- added joint 9_50: type revolute, parent 9, child 50, origin xyz=0.0 -0.19933864034087653 -0.1967585345493622 rpy=0 0 0, axis 1 0 0, limit lower=-3.14159 upper=3.14159 effort=0.0 velocity=0.0
- added joint 9_51: type revolute, parent 9, child 51, origin xyz=0.0 0.0 -0.3603917300681739 rpy=0 0 0, axis 0 1 0, limit lower=-3.14159 upper=3.14159 effort=0.0 velocity=0.0
- joint 0_1: axis 0 1 0 -> 0 0 1; origin xyz=0.0 0.0 0.15216761881022012 rpy=0 0 0 -> xyz=0.0 -0.1978379149980429 5.0 rpy=0 0 0
- joint 10_11: axis 0 1 0 -> 1 0 0; origin xyz=0.26976220716469335 0.16402130395654313 0.0 rpy=0 0 0 -> xyz=0.0 -0.2501426365879886 0.0 rpy=0 0 0
- joint 1_2: axis 0 1 0 -> 1 0 0; origin xyz=0.0 0.0 0.41981447219636553 rpy=0 0 0 -> xyz=0.0 -0.3745064011564245 0.0 rpy=0 0 0
- joint 2_3: axis 1 0 0 -> 0 0 1; origin xyz=0.0 0.0 0.4677023037709393 rpy=0 0 0 -> xyz=0.0 -0.5487095567140214 0.0 rpy=0 0 0
- joint 3_4: axis 0 1 0 -> 0 0 1; origin xyz=0.22791596911894796 0.0 0.1701979308014471 rpy=0 0 0 -> xyz=0.0 -0.4015055511376921 0.0 rpy=0 0 0
- joint 4_5: axis 0 1 0 -> 1 0 0; origin xyz=0.48238450993940946 0.0 0.0 rpy=0 0 0 -> xyz=0.0 -0.7308539585711095 0.0 rpy=0 0 0
- joint 5_6: origin xyz=0.1879151298134637 0.23933812726198045 0.0 rpy=0 0 0 -> xyz=0.0 -0.4556929607867905 0.0 rpy=0 0 0
- joint 6_7: axis 1 0 0 -> 0 0 1; origin xyz=0.0 0.4835471362875196 0.0 rpy=0 0 0 -> xyz=0.0 -0.31509732215680475 0.0 rpy=0 0 0
- joint 7_8: axis 0 1 0 -> 0 0 1; origin xyz=0.2081441937844638 0.1466280206098742 0.0 rpy=0 0 0 -> xyz=0.0 -0.7373642221112688 0.0 rpy=0 0 0
- joint 8_9: axis 0 1 0 -> 1 0 0; origin xyz=0.15707230717314155 0.0 0.26415229301022625 rpy=0 0 0 -> xyz=0.0 -0.5900883511200627 0.0 rpy=0 0 0
- joint 9_10: axis 0 0 1 -> 1 0 0; origin xyz=0.0 0.21080032869381593 0.3009367114199696 rpy=0 0 0 -> xyz=0.0 -0.39867728068175307 0.0 rpy=0 0 0
