Commit message: Minor bug fix

File: horse.urdf (robot description, URDF)
Before this commit: robot robot, 55 links, 54 joints
Links:
- removed link 10
- removed link 11
- removed link 12
- removed link 13
- removed link 14
- removed link 15
- removed link 16
- removed link 17
- removed link 18
- removed link 19
- removed link 20
- removed link 21
- removed link 22
- removed link 23
- removed link 24
- removed link 25
- removed link 26
- removed link 27
- removed link 28
- removed link 29
- removed link 30
- removed link 31
- removed link 32
- removed link 33
- removed link 34
- removed link 35
- removed link 36
- removed link 37
- removed link 38
- removed link 39
- removed link 40
- removed link 41
- removed link 42
- removed link 43
- removed link 44
- removed link 45
- removed link 46
- removed link 47
- removed link 48
- removed link 49
- removed link 50
- removed link 51
- removed link 52
- removed link 53
- removed link 54
- removed link 7
- removed link 8
- removed link 9
- link 0: geometry collision box size=0.2647244944067496 0.6461102488840818 0.5664653602495617; visual box size=0.2647244944067496 0.6461102488840818 0.5664653602495617
- link 1: geometry collision box size=0.3984609017084142 0.5648388540539568 0.4785178917875639; visual box size=0.3984609017084142 0.5648388540539568 0.4785178917875639
- link 2: geometry collision box size=0.37024302276381005 0.6061813236367808 0.36011638085112274; visual box size=0.37024302276381005 0.6061813236367808 0.36011638085112274
- link 3: geometry collision box size=0.4910881957859852 0.7084479131907623 0.5479754937242818; visual box size=0.4910881957859852 0.7084479131907623 0.5479754937242818
- link 4: geometry collision box size=0.6356451477384688 0.7255384357026723 0.3213239122016431; visual box size=0.6356451477384688 0.7255384357026723 0.3213239122016431
- link 5: geometry collision box size=0.45491367471656474 0.5533069975378826 0.6605868370434149; visual box size=0.45491367471656474 0.5533069975378826 0.6605868370434149
- link 6: geometry collision box size=0.3699912068059852 0.488278540210975 0.5813646684707059; visual box size=0.3699912068059852 0.488278540210975 0.5813646684707059
Joints:
- removed joint 10_11
- removed joint 10_52
- removed joint 10_53
- removed joint 10_54
- removed joint 1_2
- removed joint 2_12
- removed joint 2_13
- removed joint 2_14
- removed joint 2_15
- removed joint 2_16
- removed joint 2_3
- removed joint 3_4
- removed joint 4_17
- removed joint 4_18
- removed joint 4_19
- removed joint 4_20
- removed joint 4_5
- removed joint 5_21
- removed joint 5_22
- removed joint 5_23
- removed joint 5_24
- removed joint 5_25
- removed joint 5_26
- removed joint 5_27
- removed joint 5_6
- removed joint 6_28
- removed joint 6_29
- removed joint 6_30
- removed joint 6_31
- removed joint 6_32
- removed joint 6_7
- removed joint 7_33
- removed joint 7_34
- removed joint 7_35
- removed joint 7_36
- removed joint 7_37
- removed joint 7_8
- removed joint 8_38
- removed joint 8_39
- removed joint 8_40
- removed joint 8_41
- removed joint 8_42
- removed joint 8_43
- removed joint 8_44
- removed joint 8_9
- removed joint 9_10
- removed joint 9_45
- removed joint 9_46
- removed joint 9_47
- removed joint 9_48
- removed joint 9_49
- removed joint 9_50
- removed joint 9_51
- added joint 0_2: type revolute, parent 0, child 2, origin xyz=0.0 0.3230551244420409 5.0 rpy=0 0 0, axis 1 0 0, limit lower=-3.14159 upper=3.14159 effort=0.0 velocity=0.0
- added joint 0_3: type revolute, parent 0, child 3, origin xyz=0.0 0.6061813236367808 0.0 rpy=0 0 0, axis 0 0 1, limit lower=-3.14159 upper=3.14159 effort=0.0 velocity=0.0
- added joint 0_4: type revolute, parent 0, child 4, origin xyz=0.0 0.7084479131907623 0.0 rpy=0 0 0, axis 0 0 1, limit lower=-3.14159 upper=3.14159 effort=0.0 velocity=0.0
- added joint 0_5: type revolute, parent 0, child 5, origin xyz=0.0 0.7255384357026723 0.0 rpy=0 0 0, axis 1 0 0, limit lower=-3.14159 upper=3.14159 effort=0.0 velocity=0.0
- added joint 1_6: type revolute, parent 1, child 6, origin xyz=0.0 0.2824194270269784 -0.23925894589378194 rpy=0 0 0, axis 0 0 1, limit lower=-3.14159 upper=3.14159 effort=0.0 velocity=0.0
- joint 0_1: axis 0 0 1 -> 1 0 0; origin xyz=0.0 -0.1978379149980429 5.0 rpy=0 0 0 -> xyz=0.0 0.0 4.716767319875219 rpy=0 0 0

Commit message: Could not debug limb issue :(

File: horse.urdf (robot description, URDF)
Before this commit: robot robot, 7 links, 6 joints
Links:
- added link 10, mass 1; collision box size=0.6241253838250692 0.5564078380437367 0.6270774131260213; visual box size=0.6241253838250692 0.5564078380437367 0.6270774131260213
- added link 7, mass 1; collision box size=0.37865772677021065 0.5421300018797814 0.7037138037204831; visual box size=0.37865772677021065 0.5421300018797814 0.7037138037204831
- added link 8, mass 1; collision box size=0.5925138821570723 0.38384267682990997 0.4286333260089051; visual box size=0.5925138821570723 0.38384267682990997 0.4286333260089051
- added link 9, mass 1; collision box size=0.540430961613331 0.6681772540047142 0.7211788840931408; visual box size=0.540430961613331 0.6681772540047142 0.7211788840931408
- link 0: geometry collision box size=0.6922211442329889 0.7223478616698422 0.49822911081857735; visual box size=0.6922211442329889 0.7223478616698422 0.49822911081857735
- link 1: geometry collision box size=0.4246263139693574 0.7275661590326445 0.66478972745211; visual box size=0.4246263139693574 0.7275661590326445 0.66478972745211
- link 2: geometry collision box size=0.28574540227291156 0.6144007544732322 0.7138184607576912; visual box size=0.28574540227291156 0.6144007544732322 0.7138184607576912
- link 3: geometry collision box size=0.35139631200949606 0.5840566008444273 0.7097561920306478; visual box size=0.35139631200949606 0.5840566008444273 0.7097561920306478
- link 4: geometry collision box size=0.6701419692726199 0.7059259719808286 0.4373954283695172; visual box size=0.6701419692726199 0.7059259719808286 0.4373954283695172
- link 5: geometry collision box size=0.527651033511465 0.44059253974213386 0.3152845606850825; visual box size=0.527651033511465 0.44059253974213386 0.3152845606850825
- link 6: geometry collision box size=0.5865549832155086 0.6098050611734672 0.2748410740417342; visual box size=0.5865549832155086 0.6098050611734672 0.2748410740417342
Joints:
- removed joint 0_2
- removed joint 0_3
- removed joint 0_4
- removed joint 0_5
- added joint 1_2: type revolute, parent 1, child 2, origin xyz=0.4246263139693574 0.0 0.0 rpy=0 0 0, axis 0 1 0, limit lower=-3.14159 upper=3.14159 effort=0.0 velocity=0.0
- added joint 1_5: type revolute, parent 1, child 5, origin xyz=0.2123131569846787 0.0 0.332394863726055 rpy=0 0 0, axis 1 0 0, limit lower=-3.14159 upper=3.14159 effort=0.0 velocity=0.0
- added joint 1_7: type revolute, parent 1, child 7, origin xyz=0.0 0.0 0.2748410740417342 rpy=0 0 0, axis 0 1 0, limit lower=-3.14159 upper=3.14159 effort=0.0 velocity=0.0
- added joint 2_10: type revolute, parent 2, child 10, origin xyz=0.0 0.0 0.7211788840931408 rpy=0 0 0, axis 1 0 0, limit lower=-3.14159 upper=3.14159 effort=0.0 velocity=0.0
- added joint 2_3: type revolute, parent 2, child 3, origin xyz=0.28574540227291156 0.0 0.0 rpy=0 0 0, axis 0 1 0, limit lower=-3.14159 upper=3.14159 effort=0.0 velocity=0.0
- added joint 2_8: type revolute, parent 2, child 8, origin xyz=0.14287270113645578 0.0 0.3569092303788456 rpy=0 0 0, axis 0 1 0, limit lower=-3.14159 upper=3.14159 effort=0.0 velocity=0.0
- added joint 2_9: type revolute, parent 2, child 9, origin xyz=0.0 0.0 0.4286333260089051 rpy=0 0 0, axis 1 0 0, limit lower=-3.14159 upper=3.14159 effort=0.0 velocity=0.0
- added joint 3_4: type revolute, parent 3, child 4, origin xyz=0.35139631200949606 0.0 0.0 rpy=0 0 0, axis 0 1 0, limit lower=-3.14159 upper=3.14159 effort=0.0 velocity=0.0
- joint 0_1: axis 1 0 0 -> 0 1 0; origin xyz=0.0 0.0 4.716767319875219 rpy=0 0 0 -> xyz=0.34611057211649443 0.0 5.0 rpy=0 0 0
- joint 1_6: axis 0 0 1 -> 1 0 0; origin xyz=0.0 0.2824194270269784 -0.23925894589378194 rpy=0 0 0 -> xyz=0.0 0.0 0.3152845606850825 rpy=0 0 0

Commit message: Fixed Construct_Limb()

File: horse.urdf (robot description, URDF)
Before this commit: robot robot, 11 links, 10 joints
Links:
- added link 11, mass 1; collision box size=0.41207050389660704 0.3248374335918416 0.3611606941257938; visual box size=0.41207050389660704 0.3248374335918416 0.3611606941257938
- added link 12, mass 1; collision box size=0.44324449056293097 0.7012992377647023 0.4749749949556138; visual box size=0.44324449056293097 0.7012992377647023 0.4749749949556138
- added link 13, mass 1; collision box size=0.5565317289420662 0.7011742915869921 0.29964017517948693; visual box size=0.5565317289420662 0.7011742915869921 0.29964017517948693
- added link 14, mass 1; collision box size=0.7349045338733744 0.5765700178989688 0.3354547925680226; visual box size=0.7349045338733744 0.5765700178989688 0.3354547925680226
- link 0: geometry collision box size=0.75 0.75 0.75; visual box size=0.75 0.75 0.75
- link 1: geometry collision box size=0.75 0.75 0.75; visual box size=0.75 0.75 0.75
- link 10: geometry collision box size=0.6184590885644791 0.35827517721218594 0.31760908670272603; visual box size=0.6184590885644791 0.35827517721218594 0.31760908670272603
- link 2: geometry collision box size=0.75 0.75 0.75; visual box size=0.75 0.75 0.75
- link 3: geometry collision box size=0.6560843643877465 0.48998858618752866 0.44639239805041486; visual box size=0.6560843643877465 0.48998858618752866 0.44639239805041486
- link 4: geometry collision box size=0.6680393817686887 0.4186980802086342 0.5740859360255985; visual box size=0.6680393817686887 0.4186980802086342 0.5740859360255985
- link 5: geometry collision box size=0.434120769920274 0.7285775794765232 0.3201753902063226; visual box size=0.434120769920274 0.7285775794765232 0.3201753902063226
- link 6: geometry collision box size=0.6850436291792181 0.48680402263685524 0.6504553759898222; visual box size=0.6850436291792181 0.48680402263685524 0.6504553759898222
- link 7: geometry collision box size=0.5102387397756024 0.5894397650594801 0.6103163273629584; visual box size=0.5102387397756024 0.5894397650594801 0.6103163273629584
- link 8: geometry collision box size=0.5410098960375536 0.5186866147245053 0.6293078121611786; visual box size=0.5410098960375536 0.5186866147245053 0.6293078121611786
- link 9: geometry collision box size=0.30295380359389606 0.4868002096733287 0.34316617166338; visual box size=0.30295380359389606 0.4868002096733287 0.34316617166338
Joints:
- removed joint 1_5
- removed joint 1_6
- removed joint 1_7
- removed joint 2_10
- removed joint 2_3
- removed joint 2_8
- removed joint 2_9
- added joint 0_3: type revolute, parent 0, child 3, origin xyz=0.0 0.375 5.0 rpy=0 0 0, axis 0 0 1, limit lower=-3.14159 upper=3.14159 effort=0.0 velocity=0.0
- added joint 0_5: type revolute, parent 0, child 5, origin xyz=0.0 -0.375 5.0 rpy=0 0 0, axis 0 0 1, limit lower=-3.14159 upper=3.14159 effort=0.0 velocity=0.0
- added joint 11_12: type revolute, parent 11, child 12, origin xyz=0.0 0.0 0.3611606941257938 rpy=0 0 0, axis 1 0 0, limit lower=-3.14159 upper=3.14159 effort=0.0 velocity=0.0
- added joint 13_14: type revolute, parent 13, child 14, origin xyz=0.0 0.0 -0.29964017517948693 rpy=0 0 0, axis 0 1 0, limit lower=-3.14159 upper=3.14159 effort=0.0 velocity=0.0
- added joint 1_8: type revolute, parent 1, child 8, origin xyz=0.375 0.0 -0.375 rpy=0 0 0, axis 1 0 0, limit lower=-3.14159 upper=3.14159 effort=0.0 velocity=0.0
- added joint 2_11: type revolute, parent 2, child 11, origin xyz=0.375 0.0 0.375 rpy=0 0 0, axis 0 1 0, limit lower=-3.14159 upper=3.14159 effort=0.0 velocity=0.0
- added joint 2_13: type revolute, parent 2, child 13, origin xyz=0.375 0.0 -0.375 rpy=0 0 0, axis 0 1 0, limit lower=-3.14159 upper=3.14159 effort=0.0 velocity=0.0
- added joint 5_6: type revolute, parent 5, child 6, origin xyz=0.0 -0.7285775794765232 0.0 rpy=0 0 0, axis 1 0 0, limit lower=-3.14159 upper=3.14159 effort=0.0 velocity=0.0
- added joint 6_7: type revolute, parent 6, child 7, origin xyz=0.0 -0.48680402263685524 0.0 rpy=0 0 0, axis 1 0 0, limit lower=-3.14159 upper=3.14159 effort=0.0 velocity=0.0
- added joint 8_9: type revolute, parent 8, child 9, origin xyz=0.0 0.0 -0.6293078121611786 rpy=0 0 0, axis 0 1 0, limit lower=-3.14159 upper=3.14159 effort=0.0 velocity=0.0
- added joint 9_10: type revolute, parent 9, child 10, origin xyz=0.0 0.0 -0.34316617166338 rpy=0 0 0, axis 1 0 0, limit lower=-3.14159 upper=3.14159 effort=0.0 velocity=0.0
- joint 0_1: axis 0 1 0 -> 0 0 1; origin xyz=0.34611057211649443 0.0 5.0 rpy=0 0 0 -> xyz=0.375 0.0 5.0 rpy=0 0 0
- joint 1_2: axis 0 1 0 -> 0 0 1; origin xyz=0.4246263139693574 0.0 0.0 rpy=0 0 0 -> xyz=0.75 0.0 0.0 rpy=0 0 0
- joint 3_4: axis 0 1 0 -> 0 0 1; origin xyz=0.35139631200949606 0.0 0.0 rpy=0 0 0 -> xyz=0.0 0.48998858618752866 0.0 rpy=0 0 0

Commit message: Fixed bugs to fill space

File: horse.urdf (robot description, URDF)
Before this commit: robot robot, 15 links, 14 joints
Links:
- removed link 10
- removed link 11
- removed link 12
- removed link 13
- removed link 14
- link 3: geometry collision box size=0.75 0.75 0.75; visual box size=0.75 0.75 0.75
- link 4: geometry collision box size=0.5740859360255985 0.434120769920274 0.7285775794765232; visual box size=0.5740859360255985 0.434120769920274 0.7285775794765232
- link 5: geometry collision box size=0.26315785118569035 0.5915392662612964 0.41312362037316974; visual box size=0.26315785118569035 0.5915392662612964 0.41312362037316974
- link 6: geometry collision box size=0.47036430079185776 0.358190991820482 0.4215518120475841; visual box size=0.47036430079185776 0.358190991820482 0.4215518120475841
- link 7: geometry collision box size=0.569960510663762 0.3216766437045232 0.722334458524792; visual box size=0.569960510663762 0.3216766437045232 0.722334458524792
- link 8: geometry collision box size=0.4573309699952618 0.3822778060523135 0.6371168447171083; visual box size=0.4573309699952618 0.3822778060523135 0.6371168447171083
- link 9: geometry collision box size=0.40526764949744687 0.45579527699089184 0.20845541019635982; visual box size=0.40526764949744687 0.45579527699089184 0.20845541019635982
Joints:
- removed joint 0_3
- removed joint 0_5
- removed joint 11_12
- removed joint 13_14
- removed joint 1_8
- removed joint 2_11
- removed joint 2_13
- removed joint 3_4
- removed joint 6_7
- removed joint 9_10
- added joint 1_4: type revolute, parent 1, child 4, origin xyz=0.375 0.0 0.375 rpy=0 0 0, axis 1 0 0, limit lower=-3.14159 upper=3.14159 effort=0.0 velocity=0.0
- added joint 2_3: type revolute, parent 2, child 3, origin xyz=0.75 0.0 0.0 rpy=0 0 0, axis 0 0 1, limit lower=-3.14159 upper=3.14159 effort=0.0 velocity=0.0
- added joint 2_7: type revolute, parent 2, child 7, origin xyz=0.375 0.0 -0.375 rpy=0 0 0, axis 1 0 0, limit lower=-3.14159 upper=3.14159 effort=0.0 velocity=0.0
- added joint 3_8: type revolute, parent 3, child 8, origin xyz=0.375 0.0 -0.375 rpy=0 0 0, axis 1 0 0, limit lower=-3.14159 upper=3.14159 effort=0.0 velocity=0.0
- added joint 4_5: type revolute, parent 4, child 5, origin xyz=0.0 0.217060384960137 0.3642887897382616 rpy=0 0 0, axis 0 0 1, limit lower=-3.14159 upper=3.14159 effort=0.0 velocity=0.0
- joint 1_2: axis 0 0 1 -> 0 1 0
- joint 5_6: axis 1 0 0 -> 0 1 0; origin xyz=0.0 -0.7285775794765232 0.0 rpy=0 0 0 -> xyz=0.0 0.2957696331306482 0.20656181018658487 rpy=0 0 0
- joint 8_9: axis 0 1 0 -> 1 0 0; origin xyz=0.0 0.0 -0.6293078121611786 rpy=0 0 0 -> xyz=0.0 -0.19113890302615674 -0.31855842235855414 rpy=0 0 0
